File: Schaltungen/Gleisbesetzmeldung.brd (EAGLE design)
At the start: 88 parts, among them IC1 CNY-17-2, IC2 CNY-17-2, IC3 CNY-17-2, IC4 CNY-17-2, IC5 CNY-17-2, IC6 CNY-17-2, IC7 CNY-17-2, IC8 CNY-17-2

Commit message: update
Routing:
- net S$119: track 9.19 -> 13.0 mm
- net S$103: track 9.19 -> 13.0 mm
- net S$87: track 9.19 -> 13.0 mm
- net S$79: track 9.19 -> 13.0 mm
- net S$71: track 9.19 -> 13.0 mm
- net S$3: track 9.19 -> 13.0 mm
- net S$95: track 9.19 -> 13.0 mm
- net S$111: track 9.19 -> 13.0 mm
Other:
- board text added: "+"
- board text added: "-"
- board text added: "5V"
- board text added: "S0"
Changed lines of the file:
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@@
 <rectangle x1="72.39" y1="44.45" x2="73.66" y2="48.26" layer="16"/>
 <rectangle x1="83.82" y1="44.45" x2="85.09" y2="48.26" layer="16"/>
+<text x="10.16" y="3.81" size="1.27" layer="16" rot="MR0">5V</text>
+<text x="21.59" y="3.81" size="1.27" layer="16" rot="MR0">5V</text>
+<text x="33.02" y="3.81" size="1.27" layer="16" rot="MR0">5V</text>
+<text x="44.45" y="3.81" size="1.27" layer="16" rot="MR0">5V</text>
+<text x="55.88" y="3.81" size="1.27" layer="16" rot="MR0">5V</text>
+<text x="67.31" y="3.81" size="1.27" layer="16" rot="MR0">5V</text>
+<text x="78.74" y="3.81" size="1.27" layer="16" rot="MR0">5V</text>
+<text x="90.17" y="3.81" size="1.27" layer="16" rot="MR0">5V</text>
+<text x="8.89" y="53.34" size="1.27" layer="16" rot="MR0">+</text>
+<text x="20.32" y="53.34" size="1.27" layer="16" rot="MR0">+</text>
+<text x="31.75" y="53.34" size="1.27" layer="16" rot="MR0">+</text>
+<text x="43.18" y="53.34" size="1.27" layer="16" rot="MR0">+</text>
+<text x="54.61" y="53.34" size="1.27" layer="16" rot="MR0">+</text>
+<text x="66.04" y="53.34" size="1.27" layer="16" rot="MR0">+</text>
+<text x="77.47" y="53.34" size="1.27" layer="16" rot="MR0">+</text>
+<text x="88.9" y="53.34" size="1.27" layer="16" rot="MR0">+</text>
+<text x="1.27" y="0" size="1.27" layer="16" rot="MR0">-</text>
+<text x="12.7" y="0" size="1.27" layer="16" rot="MR0">-</text>
+<text x="24.13" y="0" size="1.27" layer="16" rot="MR0">-</text>
+<text x="35.56" y="0" size="1.27" layer="16" rot="MR0">-</text>
+<text x="46.99" y="0" size="1.27" layer="16" rot="MR0">-</text>
+<text x="58.42" y="0" size="1.27" layer="16" rot="MR0">-</text>
+<text x="69.85" y="0" size="1.27" layer="16" rot="MR0">-</text>
+<text x="81.28" y="0" size="1.27" layer="16" rot="MR0">-</text>
+<text x="5.08" y="0" size="0.6096" layer="16" rot="MR0">S0</text>
+<text x="27.94" y="0" size="0.6096" layer="16" rot="MR0">S0</text>
+<text x="39.37" y="0" size="0.6096" layer="16" rot="MR0">S0</text>
+<text x="50.8" y="0" size="0.6096" layer="16" rot="MR0">S0</text>
+<text x="62.23" y="0" size="0.6096" layer="16" rot="MR0">S0</text>
+<text x="73.66" y="0" size="0.6096" layer="16" rot="MR0">S0</text>
+<text x="85.09" y="0" size="0.6096" layer="16" rot="MR0">S0</text>
+<rectangle x1="1.27" y1="11.43" x2="2.54" y2="21.59" layer="16"/>
+<rectangle x1="12.7" y1="11.43" x2="13.97" y2="21.59" layer="16"/>
+<rectangle x1="24.13" y1="11.43" x2="25.4" y2="21.59" layer="16"/>
+<rectangle x1="35.56" y1="11.43" x2="36.83" y2="21.59" layer="16"/>
+<rectangle x1="46.99" y1="11.43" x2="48.26" y2="21.59" layer="16"/>
+<rectangle x1="58.42" y1="11.43" x2="59.69" y2="21.59" layer="16"/>
+<rectangle x1="69.85" y1="11.43" x2="71.12" y2="21.59" layer="16"/>
+<rectangle x1="81.28" y1="11.43" x2="82.55" y2="21.59" layer="16"/>
 </plain>
 <attributes>
@@
 <wire x1="8.89" y1="11.43" x2="7.62" y2="8.89" width="0.6096" layer="16"/>
 <wire x1="7.62" y1="8.89" x2="7.62" y2="2.54" width="1.27" layer="16"/>
+<wire x1="8.89" y1="11.43" x2="7.62" y2="11.43" width="1.27" layer="16"/>
+<wire x1="7.62" y1="11.43" x2="7.62" y2="8.89" width="1.27" layer="16"/>
 </signal>
 <signal name="S$4">
@@
 <wire x1="20.32" y1="11.43" x2="19.05" y2="8.89" width="0.6096" layer="16"/>
 <wire x1="19.05" y1="8.89" x2="19.05" y2="2.54" width="1.27" layer="16"/>
+<wire x1="20.32" y1="11.43" x2="19.05" y2="11.43" width="1.27" layer="16"/>
+<wire x1="19.05" y1="11.43" x2="19.05" y2="8.89" width="1.27" layer="16"/>
 </signal>
 <signal name="S$72">
@@
 <wire x1="31.75" y1="11.43" x2="30.48" y2="8.89" width="0.6096" layer="16"/>
 <wire x1="30.48" y1="8.89" x2="30.48" y2="2.54" width="1.27" layer="16"/>
+<wire x1="31.75" y1="11.43" x2="30.48" y2="11.43" width="1.27" layer="16"/>
+<wire x1="30.48" y1="11.43" x2="30.48" y2="8.89" width="1.27" layer="16"/>
 </signal>
 <signal name="S$80">
@@
 <wire x1="43.18" y1="11.43" x2="41.91" y2="8.89" width="0.6096" layer="16"/>
 <wire x1="41.91" y1="8.89" x2="41.91" y2="2.54" width="1.27" layer="16"/>
+<wire x1="43.18" y1="11.43" x2="41.91" y2="11.43" width="1.27" layer="16"/>
+<wire x1="41.91" y1="11.43" x2="41.91" y2="8.89" width="1.27" layer="16"/>
 </signal>
 <signal name="S$88">
@@
 <wire x1="54.61" y1="11.43" x2="53.34" y2="8.89" width="0.6096" layer="16"/>
 <wire x1="53.34" y1="8.89" x2="53.34" y2="2.54" width="1.27" layer="16"/>
+<wire x1="54.61" y1="11.43" x2="53.34" y2="11.43" width="1.27" layer="16"/>
+<wire x1="53.34" y1="11.43" x2="53.34" y2="8.89" width="1.27" layer="16"/>
 </signal>
 <signal name="S$96">
@@
 <wire x1="66.04" y1="11.43" x2="64.77" y2="8.89" width="0.6096" layer="16"/>
 <wire x1="64.77" y1="8.89" x2="64.77" y2="2.54" width="1.27" layer="16"/>
+<wire x1="66.04" y1="11.43" x2="64.77" y2="11.43" width="1.27" layer="16"/>
+<wire x1="64.77" y1="11.43" x2="64.77" y2="8.89" width="1.27" layer="16"/>
 </signal>
 <signal name="S$104">
@@
 <wire x1="77.47" y1="11.43" x2="76.2" y2="8.89" width="0.6096" layer="16"/>
 <wire x1="76.2" y1="8.89" x2="76.2" y2="2.54" width="1.27" layer="16"/>
+<wire x1="77.47" y1="11.43" x2="76.2" y2="11.43" width="1.27" layer="16"/>
+<wire x1="76.2" y1="11.43" x2="76.2" y2="8.89" width="1.27" layer="16"/>
 </signal>
 <signal name="S$112">
@@
 <wire x1="88.9" y1="11.43" x2="87.63" y2="8.89" width="0.6096" layer="16"/>
 <wire x1="87.63" y1="8.89" x2="87.63" y2="2.54" width="1.27" layer="16"/>
+<wire x1="88.9" y1="11.43" x2="87.63" y2="11.43" width="1.27" layer="16"/>
+<wire x1="87.63" y1="11.43" x2="87.63" y2="8.89" width="1.27" layer="16"/>
 </signal>
 <signal name="S$120">
