File: Schaltungen/DCC2Arduino2.brd (EAGLE design)
At the start: 84 parts, among them IC1 6N137, IC10 6N137, IC11 6N137, IC12 6N137, IC2 6N137, IC3 6N137, IC4 6N137, IC5 6N137, IC6 6N137, IC7 6N137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

Commit message: update
Other:
- board text removed: "www.cbries.de"
Changed lines of the file:
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@@
 <drawing>
 <settings>
-<setting alwaysvectorfont="no"/>
+<setting alwaysvectorfont="yes"/>
 <setting verticaltext="up"/>
 </settings>
@@
 <text x="114.935" y="11.43" size="0.4064" layer="16" rot="MR270">+</text>
 <text x="109.855" y="11.43" size="0.4064" layer="16" rot="MR270">-</text>
-<text x="27.305" y="42.545" size="1.016" layer="16" rot="MR0">www.cbries.de</text>
-<text x="66.04" y="42.545" size="1.016" layer="16" rot="MR0">www.cbries.de</text>
-<text x="104.775" y="42.545" size="1.016" layer="16" rot="MR0">www.cbries.de</text>
-<text x="104.775" y="27.94" size="1.016" layer="16" rot="MR0">www.cbries.de</text>
-<text x="104.775" y="13.335" size="1.016" layer="16" rot="MR0">www.cbries.de</text>
-<text x="109.855" y="9.525" size="1.016" layer="16" rot="MR0">www.cbries.de</text>
-<text x="88.265" y="11.43" size="1.016" layer="16" rot="MR0">www.cbries.de</text>
-<text x="48.895" y="11.43" size="1.016" layer="16" rot="MR0">www.cbries.de</text>
-<text x="10.16" y="11.43" size="1.016" layer="16" rot="MR0">www.cbries.de</text>
-<text x="26.67" y="13.335" size="1.016" layer="16" rot="MR0">www.cbries.de</text>
-<text x="65.405" y="13.335" size="1.016" layer="16" rot="MR0">www.cbries.de</text>
-<text x="65.405" y="27.94" size="1.016" layer="16" rot="MR0">www.cbries.de</text>
-<text x="26.67" y="27.94" size="1.016" layer="16" rot="MR0">www.cbries.de</text>
 </plain>
 <attributes>
