File: Schaltungen/Gleisbesetzmeldung3.brd (EAGLE design)
At the start: 13 parts, among them IC1 CNY-17-2

Commit message: update
Parts:
- removed D0, D1, D2, D3: (no value), diode:D-2.5
- added C2, C3, C4, C5, C6, C7, C8: 22uF, 35V, rcl:E2,5-5
- added E$10, E$12, E$14, E$16, E$4, E$6, E$8: (no value), led:LED3MM
- added E$11, E$13, E$15, E$17, E$5, E$7, E$9: (no value), pinhead:1X02
- added IC10, IC12, IC14, IC16, IC2, IC4, IC6, IC8: S462, rectifier:RB1A
- added IC11, IC13, IC15, IC3, IC5, IC7, IC9: CNY-17-2, ic-package:DIL06
- added P1, P3, P4, P5, P6, P7, P8: (no value), con-lstb:MA03-1
- added R10, R11, R13, R14, R16, R17, R19, R20, R22, R23, R4, R5, R7, R8: 1k, rcl:0204/7
- added R12, R15, R18, R21, R24, R6, R9: 220, rcl:0204/7
- added T2, T3, T4, T5, T6, T7, T8: (no value), transistor-neu-to92:TO92-CBE
- moved E$1 10.2 mm to (9.53, 42.5), turned to 0 degrees
- moved R2 10.2 mm to (1.27, 22.9)
- moved P2 7.75 mm to (1.91, 40.6), turned to 270 degrees
- moved T1 5.71 mm to (3.81, 33.7)
- moved R3 3.81 mm to (8.89, 35.6)
- moved C1 2.84 mm to (8.89, 16.5)
- moved R1 2.54 mm to (1.27, 11.4)
- moved IC1 2.29 mm to (7.62, 24.8)
- moved E$2 1.91 mm to (3.17, 1.91)
Connections:
- removed net S$122: D2.C, D3.A
- new net S$123: P1.3, R4.1, T2.C
- new net S$124: IC3.5, IC3.6, R4.2, T2.B
- new net S$125: E$4.A, E$4.K, IC3.4, P1.1, P1.2, R6.1, R6.2, T2.E
- new net S$126: C2.-, E$5.1, E$5.2, IC3.2, IC4.-, IC4.AC1, IC4.AC2
- new net S$127: C3.+, IC6.+, R8.2
- new net S$128: IC5.1, R8.1
- new net S$129: P3.3, R7.1, T3.C
- new net S$130: IC5.5, IC5.6, R7.2, T3.B
- new net S$131: E$6.A, E$6.K, IC5.4, P3.1, P3.2, R9.1, R9.2, T3.E
- new net S$132: C3.-, E$7.1, E$7.2, IC5.2, IC6.-, IC6.AC1, IC6.AC2
- new net S$133: C4.+, IC8.+, R11.2
- new net S$134: IC7.1, R11.1
- new net S$135: P4.3, R10.1, T4.C
- new net S$136: IC7.5, IC7.6, R10.2, T4.B
- new net S$137: E$8.A, E$8.K, IC7.4, P4.1, P4.2, R12.1, R12.2, T4.E
- new net S$138: C4.-, E$9.1, E$9.2, IC7.2, IC8.-, IC8.AC1, IC8.AC2
- new net S$139: C5.+, IC10.+, R14.2
- new net S$140: IC9.1, R14.1
- new net S$141: P5.3, R13.1, T5.C
- new net S$142: IC9.5, IC9.6, R13.2, T5.B
- new net S$143: E$10.A, E$10.K, IC9.4, P5.1, P5.2, R15.1, R15.2, T5.E
- new net S$144: C5.-, E$11.1, E$11.2, IC10.-, IC10.AC1, IC10.AC2, IC9.2
- new net S$145: C6.+, IC12.+, R17.2
- new net S$146: IC11.1, R17.1
- new net S$147: P6.3, R16.1, T6.C
- new net S$148: IC11.5, IC11.6, R16.2, T6.B
- new net S$149: E$12.A, E$12.K, IC11.4, P6.1, P6.2, R18.1, R18.2, T6.E
- new net S$150: C6.-, E$13.1, E$13.2, IC11.2, IC12.-, IC12.AC1, IC12.AC2
- new net S$151: C7.+, IC14.+, R20.2
- new net S$152: IC13.1, R20.1
- new net S$153: P7.3, R19.1, T7.C
- new net S$154: IC13.5, IC13.6, R19.2, T7.B
- new net S$155: E$14.A, E$14.K, IC13.4, P7.1, P7.2, R21.1, R21.2, T7.E
- new net S$156: C7.-, E$15.1, E$15.2, IC13.2, IC14.-, IC14.AC1, IC14.AC2
- new net S$157: C8.+, IC16.+, R23.2
- new net S$158: IC15.1, R23.1
- new net S$159: P8.3, R22.1, T8.C
- new net S$160: IC15.5, IC15.6, R22.2, T8.B
- new net S$161: E$16.A, E$16.K, IC15.4, P8.1, P8.2, R24.1, R24.2, T8.E
- new net S$162: C8.-, E$17.1, E$17.2, IC15.2, IC16.-, IC16.AC1, IC16.AC2
- net S$11: now also IC3.1, R5.1; no longer E$1.K, IC1.4, P2.1, P2.2, R3.2, T1.E
- net S$2: now also C1.-, E$2.1, E$2.2, IC1.2, IC2.-, IC2.AC1, IC2.AC2; no longer D0.C, D1.A
- net S$5: now also E$1.K, IC1.4, P2.1, P2.2, R3.2, T1.E
- net S$6: now also C2.+, IC4.+, R5.2; no longer C1.-, D0.A, D2.A, IC1.2
- net S$7: now also IC2.+; no longer D1.C, D3.C
Routing:
- net S$137: track 0.00 -> 42.2 mm
- net S$143: track 0.00 -> 42.2 mm
- net S$131: track 0.00 -> 42.2 mm
- net S$149: track 0.00 -> 42.2 mm
- net S$125: track 0.00 -> 42.2 mm
- net S$161: track 0.00 -> 42.2 mm
- net S$155: track 0.00 -> 42.2 mm
- net S$5: track 1.91 -> 42.2 mm
- net S$138: track 0.00 -> 36.6 mm
- net S$150: track 0.00 -> 36.6 mm
- net S$132: track 0.00 -> 36.6 mm
- net S$126: track 0.00 -> 36.6 mm
- net S$162: track 0.00 -> 36.6 mm
- net S$156: track 0.00 -> 36.6 mm
- net S$144: track 0.00 -> 36.6 mm
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Other:
- board text removed: "www.cbries.de (2017)"

Commit message: update
Parts:
- removed P1, P2, P3, P4, P5, P6, P7, P8: (no value), con-lstb:MA03-1
- added E$18, E$19, E$20, E$21, E$22, E$23, E$24, E$25: (no value), pinhead:1X01
- added E$3: (no value), pinhead:1X02
- E$11, E$13, E$15, E$17, E$5, E$7, E$9: device pinhead:1X02 -> pinhead:1X01
- moved E$13 3.18 mm to (73.0, 1.91), turned to 0 degrees
- moved E$7 3.18 mm to (33.0, 1.91), turned to 0 degrees
- moved E$11 3.17 mm to (59.7, 1.91), turned to 0 degrees
- moved E$15 3.17 mm to (86.4, 1.91), turned to 0 degrees
- moved E$17 3.17 mm to (100.3, 1.91), turned to 0 degrees
- moved E$5 3.17 mm to (19.7, 1.91), turned to 0 degrees
- moved E$9 3.17 mm to (46.4, 1.91), turned to 0 degrees
- moved E$2 1.91 mm to (5.08, 1.91), turned to 0 degrees
Connections:
- removed net S$125: E$4.A, E$4.K, IC3.4, P1.1, P1.2, R6.1, R6.2, T2.E
- removed net S$126: C2.-, E$5.1, E$5.2, IC3.2, IC4.-, IC4.AC1, IC4.AC2
- removed net S$131: E$6.A, E$6.K, IC5.4, P3.1, P3.2, R9.1, R9.2, T3.E
- removed net S$132: C3.-, E$7.1, E$7.2, IC5.2, IC6.-, IC6.AC1, IC6.AC2
- removed net S$135: P4.3, R10.1, T4.C
- removed net S$137: E$8.A, E$8.K, IC7.4, P4.1, P4.2, R12.1, R12.2, T4.E
- removed net S$138: C4.-, E$9.1, E$9.2, IC7.2, IC8.-, IC8.AC1, IC8.AC2
- removed net S$143: E$10.A, E$10.K, IC9.4, P5.1, P5.2, R15.1, R15.2, T5.E
- removed net S$144: C5.-, E$11.1, E$11.2, IC10.-, IC10.AC1, IC10.AC2, IC9.2
- removed net S$147: P6.3, R16.1, T6.C
- removed net S$149: E$12.A, E$12.K, IC11.4, P6.1, P6.2, R18.1, R18.2, T6.E
- removed net S$150: C6.-, E$13.1, E$13.2, IC11.2, IC12.-, IC12.AC1, IC12.AC2
- removed net S$153: P7.3, R19.1, T7.C
- removed net S$155: E$14.A, E$14.K, IC13.4, P7.1, P7.2, R21.1, R21.2, T7.E
- removed net S$156: C7.-, E$15.1, E$15.2, IC13.2, IC14.-, IC14.AC1, IC14.AC2
- removed net S$159: P8.3, R22.1, T8.C
- removed net S$161: E$16.A, E$16.K, IC15.4, P8.1, P8.2, R24.1, R24.2, T8.E
- removed net S$2: C1.-, E$2.1, E$2.2, IC1.2, IC2.-, IC2.AC1, IC2.AC2
- net S$123: no longer P1.3
- net S$129: no longer P3.3
- net S$141: no longer P5.3
- net S$162: now also C1.-, C2.-, C3.-, C4.-, C5.-, C6.-, C7.-, E$11.1, E$13.1, E$15.1, E$2.1, E$2.2, E$5.1, E$7.1, E$9.1, IC1.2, IC10.-, IC10.AC1, IC10.AC2, IC11.2, IC12.-, IC12.AC1, IC12.AC2, IC13.2, IC14.-, IC14.AC1, IC14.AC2, IC2.-, IC2.AC1, IC2.AC2, IC3.2, IC4.-, IC4.AC1, IC4.AC2, IC5.2, IC6.-, IC6.AC1, IC6.AC2, IC7.2, IC8.-, IC8.AC1, IC8.AC2, IC9.2; no longer E$17.2
- net S$3: now also E$3.2, R10.1, R16.1, R19.1, R22.1, T4.C, T6.C, T7.C, T8.C; no longer P2.3
- net S$5: now also E$10.A, E$10.K, E$12.A, E$12.K, E$14.A, E$14.K, E$16.A, E$16.K, E$18.1, E$19.1, E$20.1, E$21.1, E$22.1, E$23.1, E$24.1, E$25.1, E$3.1, E$4.A, E$4.K, E$6.A, E$6.K, E$8.A, E$8.K, IC11.4, IC13.4, IC15.4, IC3.4, IC5.4, IC7.4, IC9.4, R12.1, R12.2, R15.1, R15.2, R18.1, R18.2, R21.1, R21.2, R24.1, R24.2, R6.1, R6.2, R9.1, R9.2, T2.E, T3.E, T4.E, T5.E, T6.E, T7.E, T8.E; no longer P2.1, P2.2
Routing:
- net S$5: track 42.2 -> 365.5 mm
- net S$162: track 36.6 -> 354.1 mm
- net S$3: track 11.7 -> 200.6 mm, vias 0 -> 14
- net S$137: track 42.2 -> 0.00 mm
- net S$143: track 42.2 -> 0.00 mm
- net S$131: track 42.2 -> 0.00 mm
- net S$149: track 42.2 -> 0.00 mm
- net S$125: track 42.2 -> 0.00 mm
- net S$161: track 42.2 -> 0.00 mm
- net S$155: track 42.2 -> 0.00 mm
- net S$138: track 36.6 -> 0.00 mm
- net S$2: track 36.6 -> 0.00 mm
- net S$150: track 36.6 -> 0.00 mm
- net S$132: track 36.6 -> 0.00 mm
- net S$126: track 36.6 -> 0.00 mm
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Other:
- board text removed: "+"
- board text removed: "-"
- board text removed: "5V"
- board text removed: "GND"
- board text removed: "SIGNAL"

Commit message: update
Parts:
- removed E$11, E$13, E$15, E$17, E$18, E$19, E$20, E$21, E$22, E$23, E$24, E$25: (no value), pinhead:1X01
- added E$26, E$27, E$28: (no value), con-phoenix-254:2POL254
- added E$29: (no value), con-phoenix-254:3POL254
- E$2, E$3: device pinhead:1X02 -> con-phoenix-254:2POL254
- E$5, E$7, E$9: device pinhead:1X01 -> con-phoenix-254:2POL254
- moved E$5 55.9 mm to (48.9, 49.5)
- moved E$7 52.3 mm to (54.6, 49.5)
- moved E$9 49.6 mm to (60.3, 49.5)
- moved E$2 47.0 mm to (4.45, 48.9)
- moved E$3 41.4 mm to (43.2, 49.5), turned to 0 degrees
- moved R2 7.43 mm to (3.81, 29.8)
- moved R16 6.38 mm to (68.6, 29.2)
- moved R19 6.38 mm to (81.9, 29.2)
- moved R10 6.38 mm to (41.9, 29.2)
- moved R13 6.38 mm to (55.2, 29.2)
- moved R4 6.38 mm to (15.2, 29.2)
- moved R7 6.38 mm to (28.6, 29.2)
- moved R22 6.35 mm to (95.2, 29.2)
- moved R17 5.75 mm to (68.6, 17.1)
- moved R20 5.75 mm to (81.9, 17.1)
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Connections:
- net S$130 renamed S$2
- removed net S$123: R4.1, T2.C
- removed net S$129: R7.1, T3.C
- removed net S$141: R13.1, T5.C
- removed net S$4: IC1.5, IC1.6, R2.2, T1.B
- net S$162: now also E$26.1, E$26.2, E$27.1, E$27.2, E$28.1, E$28.2, E$29.1, E$29.2, E$29.3; no longer E$11.1, E$13.1, E$15.1, E$17.1, E$2.1, E$2.2, E$5.1, E$7.1, E$9.1
- net S$3: now also E$2.2, IC1.5, IC1.6, R13.1, R2.2, R4.1, R7.1, T1.B, T2.C, T3.C, T5.C; no longer E$3.2
- net S$5: now also E$2.1, E$3.2, E$5.1, E$5.2, E$7.1, E$7.2, E$9.1, E$9.2; no longer E$18.1, E$19.1, E$20.1, E$21.1, E$22.1, E$23.1, E$24.1, E$25.1
Routing:
- net S$5: track 365.5 -> 605.7 mm
- net S$3: track 200.6 -> 409.2 mm, vias 14 -> 0
- net S$162: track 354.1 -> 552.3 mm
- net S$4: track 20.1 -> 0.00 mm
- net S$141: track 18.4 -> 0.00 mm
- net S$129: track 18.4 -> 0.00 mm
- net S$123: track 6.98 -> 0.00 mm
- net S$2: track 20.1 -> 16.4 mm
- net S$160: track 20.1 -> 16.7 mm
- net S$154: track 20.1 -> 17.1 mm
- net S$136: track 20.1 -> 17.1 mm
- net S$124: track 20.1 -> 17.1 mm
- net S$142: track 20.1 -> 17.1 mm
- net S$148: track 20.1 -> 17.1 mm
- net S$1: track 313.7 -> 316.2 mm
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Other:
- board text added: "+"
- board text added: "-"
- board text added: "5V"
- board text added: "AREF"
- board text added: "S88 Rückmeldung"
- board text added: "www.cbries.de (03.2017)"

Commit message: update
Changed lines of the file:
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@@
 <grid distance="0.635" unitdist="mm" unit="mm" style="lines" multiple="1" display="yes" altdistance="1.27" altunitdist="mm" altunit="mm"/>
 <layers>
-<layer number="1" name="Top" color="4" fill="1" visible="yes" active="yes"/>
+<layer number="1" name="Top" color="4" fill="1" visible="no" active="yes"/>
 <layer number="16" name="Bottom" color="1" fill="1" visible="yes" active="yes"/>
 <layer number="17" name="Pads" color="2" fill="1" visible="yes" active="yes"/>
@@
 <wire x1="3.81" y1="33.655" x2="4.445" y2="34.925" width="0.6096" layer="16"/>
 <wire x1="4.445" y1="34.925" x2="4.445" y2="35.56" width="0.6096" layer="16"/>
-<wire x1="2.54" y1="45.72" x2="2.54" y2="36.83" width="0.6096" layer="16"/>
+<wire x1="2.54" y1="44.45" x2="2.54" y2="36.83" width="0.6096" layer="16"/>
 <contactref element="R2" pad="2"/>
 <contactref element="IC1" pad="6"/>
@@
 <wire x1="6.985" y1="30.48" x2="8.89" y2="31.115" width="0" layer="19" extent="16-16"/>
 <contactref element="E$2" pad="2"/>
-<wire x1="1.905" y1="45.085" x2="2.54" y2="45.72" width="0" layer="19" extent="1-16"/>
-<wire x1="2.54" y1="45.72" x2="5.715" y2="48.895" width="0.6096" layer="16"/>
+<wire x1="1.905" y1="45.085" x2="2.54" y2="44.45" width="0" layer="19" extent="1-16"/>
+<wire x1="2.54" y1="44.45" x2="5.715" y2="48.895" width="0" layer="19" extent="1-16"/>
 <wire x1="11.43" y1="44.45" x2="10.795" y2="43.815" width="0.4064" layer="16"/>
 <wire x1="10.795" y1="43.815" x2="10.16" y2="41.275" width="0" layer="19" extent="1-16"/>
+<wire x1="2.54" y1="44.45" x2="5.715" y2="47.625" width="0.6096" layer="16"/>
+<wire x1="5.715" y1="47.625" x2="5.715" y2="48.895" width="0.6096" layer="16"/>
 </signal>
 <signal name="S$9">
@@
 <wire x1="6.985" y1="25.4" x2="12.065" y2="25.4" width="0.6096" layer="16"/>
 <wire x1="12.065" y1="25.4" x2="12.065" y2="30.48" width="0.6096" layer="16"/>
-<wire x1="12.065" y1="25.4" x2="13.97" y2="22.86" width="0.6096" layer="16"/>
-<wire x1="13.97" y1="22.86" x2="16.51" y2="22.86" width="0.6096" layer="16"/>
+<wire x1="12.065" y1="25.4" x2="13.97" y2="22.86" width="0" layer="19" extent="1-16"/>
+<wire x1="13.97" y1="22.86" x2="14.605" y2="22.86" width="0" layer="19" extent="1-16"/>
+<wire x1="14.605" y1="22.86" x2="16.51" y2="22.86" width="0.6096" layer="16"/>
 <wire x1="16.51" y1="22.86" x2="19.05" y2="25.4" width="0.6096" layer="16"/>
 <wire x1="19.05" y1="25.4" x2="24.13" y2="25.4" width="0.6096" layer="16"/>
@@
 <wire x1="93.345" y1="47.625" x2="63.5" y2="47.625" width="0.4064" layer="16"/>
 <wire x1="63.5" y1="47.625" x2="61.595" y2="49.53" width="0.4064" layer="16"/>
+<wire x1="12.065" y1="25.4" x2="14.605" y2="22.86" width="0.6096" layer="16"/>
 </signal>
 <signal name="S$6">

Commit message: gerber files
Parts:
- removed E$10, E$12, E$14, E$16, E$4, E$6, E$8: (no value), led:LED3MM
- added LED2, LED3, LED4, LED5, LED6, LED7, LED8: (no value), led:LED3MM
- moved C8 7.62 mm to (95.2, 18.4)
- moved IC16 7.62 mm to (93.3, 10.8)
- moved R22 7.62 mm to (87.6, 29.2)
- moved R23 7.62 mm to (87.6, 17.1)
- moved R24 7.62 mm to (95.2, 37.5)
- moved T8 7.62 mm to (90.2, 35.6)
- moved IC15 7.62 mm to (94.0, 26.7)
- moved C7 6.98 mm to (82.5, 18.4)
- moved IC13 6.98 mm to (81.3, 26.7)
- moved IC14 6.98 mm to (80.6, 10.8)
- moved R19 6.98 mm to (74.9, 29.2)
- moved R20 6.98 mm to (74.9, 17.1)
- moved R21 6.98 mm to (82.5, 37.5)
- moved T7 6.98 mm to (77.5, 35.6)
- moved C6 5.72 mm to (70.5, 18.4)
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- renumbered E$1 to LED1, E$2 to P0, E$26 to P6, E$27 to P7, E$28 to P8, E$29 to P5, E$3 to P1, E$5 to P2, E$7 to P3, E$9 to P4
Connections:
- net S$5: now also LED2.A, LED2.K, LED3.A, LED3.K, LED4.A, LED4.K, LED5.A, LED5.K, LED6.A, LED6.K, LED7.A, LED7.K, LED8.A, LED8.K; no longer E$10.A, E$10.K, E$12.A, E$12.K, E$14.A, E$14.K, E$16.A, E$16.K, E$4.A, E$4.K, E$6.A, E$6.K, E$8.A, E$8.K
Routing:
- net S$1: track 316.2 -> 0.00 mm
- net S$162: track 552.3 -> 528.9 mm
- net S$5: track 605.5 -> 588.0 mm
- net S$3: track 409.2 -> 403.2 mm
- net S$6: track 9.57 -> 8.94 mm
- net S$11: track 4.97 -> 4.34 mm
Other:
- board outline added: 99.1 x 52.1 mm
