File: Schaltungen/LichtschrankeArduino.sch (EAGLE design)
At the start: 9 parts, among them T1 LPT80A, T2 LPT80A, T3 2N3904

Commit message: update Lichtschranke
Parts:
- C1: value (none) -> 4,7µ
- D1: value 1N4148DO35-7 -> 1N4148
- LED1: value (none) -> IRLED
- R1: value (none) -> 220
- R2: value (none) -> >47k
- R3: value (none) -> 47k
- T3: value 2N3904 -> BC337-40
Changed lines of the file:
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@@
 <setting verticaltext="up"/>
 </settings>
-<grid distance="1.27" unitdist="mm" unit="mm" style="dots" multiple="1" display="yes" altdistance="0.01" altunitdist="inch" altunit="mm"/>
+<grid distance="0.1" unitdist="inch" unit="inch" style="lines" multiple="1" display="no" altdistance="0.01" altunitdist="inch" altunit="inch"/>
 <layers>
 <layer number="1" name="Top" color="4" fill="1" visible="no" active="no"/>
@@
 </classes>
 <parts>
-<part name="C1" library="rcl" deviceset="CPOL-EU" device="E1.8-4"/>
-<part name="R1" library="rcl" deviceset="R-EU_" device="0204/2V"/>
-<part name="R2" library="rcl" deviceset="R-EU_" device="0204/2V"/>
-<part name="R3" library="rcl" deviceset="R-EU_" device="0204/2V"/>
-<part name="D1" library="diode" deviceset="1N4148" device="DO35-7"/>
-<part name="LED1" library="led" deviceset="LED" device="5MM"/>
+<part name="C1" library="rcl" deviceset="CPOL-EU" device="E1.8-4" value="4,7µ"/>
+<part name="R1" library="rcl" deviceset="R-EU_" device="0204/2V" value="220"/>
+<part name="R2" library="rcl" deviceset="R-EU_" device="0204/2V" value="&gt;47k"/>
+<part name="R3" library="rcl" deviceset="R-EU_" device="0204/2V" value="47k"/>
+<part name="D1" library="diode" deviceset="1N4148" device="DO35-7" value="1N4148"/>
+<part name="LED1" library="led" deviceset="LED" device="5MM" value="IRLED"/>
 <part name="T1" library="opto-trans-siemens" deviceset="LPT80A" device=""/>
 <part name="T2" library="opto-trans-siemens" deviceset="LPT80A" device=""/>
-<part name="T3" library="transistor" deviceset="2N3904" device=""/>
+<part name="T3" library="transistor" deviceset="2N3904" device="" value="BC337-40"/>
 </parts>
 <sheets>
